Commit message: added ros2_control for real robot

File: arns_description/urdf/ros2_control.xacro (robot description, xacro)
@@ -1,4 +1,35 @@
 <?xml version="1.0" encoding="UTF-8"?>
 <robot xmlns:xacro="http://www.ros.org/wiki/xacro">
+   <xacro:if value="$(arg sim_mode)">
+      <ros2_control name="RealRobot" type="system">
+         <hardware>
+            <plugin>diffdrive_arduino/DiffDriveArduino</plugin>
+            <param name="left_wheel_name">left_wheel_joint</param>
+            <param name="right_wheel_name">right_wheel_joint</param>
+            <param name="loop_rate">30</param>
+            <param name="device">/dev/ttyACM0</param>
+            <param name="baud_rate">57600</param>
+            <param name="timeout">1000</param>
+            <param name="enc_counts_per_rev">2800</param>
+         </hardware>
+         <joint name="left_wheel_joint">
+            <command_interface name="velocity">
+               <param name="min">-10</param>
+               <param name="max">10</param>
+            </command_interface>
+            <state_interface name="velocity"/>
+            <state_interface name="position"/>
+         </joint>
+         <joint name="right_wheel_joint">
+            <command_interface name="velocity">
+               <param name="min">-10</param>
+               <param name="max">10</param>
+            </command_interface>
+            <state_interface name="velocity"/>
+            <state_interface name="position"/>
+         </joint>
+      </ros2_control>
+   </xacro:if>
+   <xacro:if value="$(arg sim_mode)">
       <ros2_control name="GazeboSystem" type="system">
          <hardware>
@@ -22,7 +53,9 @@
          </joint>
       </ros2_control>
+   </xacro:if>
    <gazebo>
       <plugin name="gazebo_ros2_control" filename="libgazebo_ros2_control.so">
          <parameters>$(find arns_bringup)/config/controllers.yaml</parameters>
+         <parameters>$(find arns_bringup)/config/gazebo_ros2_ctl_use_sim.yaml</parameters>
       </plugin>
    </gazebo>

Commit message: fix ros2_control

File: arns_description/urdf/ros2_control.xacro (robot description, xacro)
@@ -1,33 +1,5 @@
 <?xml version="1.0" encoding="UTF-8"?>
 <robot xmlns:xacro="http://www.ros.org/wiki/xacro">
-   <ros2_control name="RealRobot" type="system">
-      <hardware>
-         <plugin>diffdrive_arduino/DiffDriveArduino</plugin>
-         <param name="left_wheel_name">left_wheel_joint</param>
-         <param name="right_wheel_name">right_wheel_joint</param>
-         <param name="loop_rate">30</param>
-         <param name="device">/dev/ttyACM0</param>
-         <param name="baud_rate">57600</param>
-         <param name="timeout">1000</param>
-         <param name="enc_counts_per_rev">2800</param>
-      </hardware>
-      <joint name="left_wheel_joint">
-         <command_interface name="velocity">
-            <param name="min">-10</param>
-            <param name="max">10</param>
-         </command_interface>
-         <state_interface name="velocity"/>
-         <state_interface name="position"/>
-      </joint>
-      <joint name="right_wheel_joint">
-         <command_interface name="velocity">
-            <param name="min">-10</param>
-            <param name="max">10</param>
-         </command_interface>
-         <state_interface name="velocity"/>
-         <state_interface name="position"/>
-      </joint>
-   </ros2_control>
-   <!-- <ros2_control name="GazeboSystem" type="system">
+   <ros2_control name="GazeboSystem" type="system">
       <hardware>
          <plugin>gazebo_ros2_control/GazeboSystem</plugin>
@@ -49,5 +21,5 @@
          <state_interface name="position"/>
       </joint>
-   </ros2_control>   -->
+   </ros2_control>
    <gazebo>
       <plugin name="gazebo_ros2_control" filename="libgazebo_ros2_control.so">

Commit message: ros2_control fixed

File: arns_description/urdf/ros2_control.xacro (robot description, xacro)
@@ -1,5 +1,33 @@
 <?xml version="1.0" encoding="UTF-8"?>
 <robot xmlns:xacro="http://www.ros.org/wiki/xacro">
-   <ros2_control name="GazeboSystem" type="system">
+   <ros2_control name="RealRobot" type="system">
+         <hardware>
+            <plugin>diffdrive_arduino/DiffDriveArduino</plugin>
+            <param name="left_wheel_name">left_wheel_joint</param>
+            <param name="right_wheel_name">right_wheel_joint</param>
+            <param name="loop_rate">30</param>
+            <param name="device">/dev/ttyACM0</param>
+            <param name="baud_rate">57600</param>
+            <param name="timeout">1000</param>
+            <param name="enc_counts_per_rev">2800</param>
+         </hardware>
+         <joint name="left_wheel_joint">
+            <command_interface name="velocity">
+               <param name="min">-10</param>
+               <param name="max">10</param>
+            </command_interface>
+            <state_interface name="velocity"/>
+            <state_interface name="position"/>
+         </joint>
+         <joint name="right_wheel_joint">
+            <command_interface name="velocity">
+               <param name="min">-10</param>
+               <param name="max">10</param>
+            </command_interface>
+            <state_interface name="velocity"/>
+            <state_interface name="position"/>
+         </joint>
+      </ros2_control>
+   <!-- <ros2_control name="GazeboSystem" type="system">
       <hardware>
          <plugin>gazebo_ros2_control/GazeboSystem</plugin>
@@ -21,5 +49,5 @@
          <state_interface name="position"/>
       </joint>
-   </ros2_control>
+   </ros2_control>   -->
    <gazebo>
       <plugin name="gazebo_ros2_control" filename="libgazebo_ros2_control.so">
