Commit message: robot_localization added

File: arns_description/urdf/robot_core.urdf.xacro (robot description, xacro)
@@ -1,13 +1,13 @@
 <?xml version="1.0" encoding="UTF-8"?>
 <robot xmlns:xacro="http://www.ros.org/wiki/xacro">
-   <link name="base_link"/>
    <!-- BASE FOOTPRINT -->
    <joint name="base_footprint_joint" type="fixed">
-      <parent link="base_link"/>
-      <child link="base_footprint"/>
+      <parent link="base_footprint"/>
+      <child link="base_link"/>
       <origin xyz="0 0 0" rpy="0 0 0"/>
    </joint>
-   <link name="base_footprint">
-   </link>
+   <link name="base_footprint"/>
+   <!-- BASE LINK -->
+   <link name="base_link"/>
    <!-- CHASSIS -->
    <joint name="chassis_joint" type="fixed">
