Commit message: first commit on branch

File: arns_description/urdf/camera.xacro (robot description, xacro)
@@ -9,5 +9,5 @@
       <visual>
          <geometry>
-            <mesh filename="file://$(find arns_description)/meshes/camera.stl" scale="0.001 0.001 0.001"/>
+            <mesh filename="file:///home/ervinpicardal/robot_ws/src/arns_description/meshes/camera.stl" scale="0.001 0.001 0.001"/>
          </geometry>
          <material name="black"/>

File: arns_description/urdf/imu.xacro (robot description, xacro)
@@ -10,5 +10,5 @@
         <origin xyz="0 0 0" rpy="0 0 ${pi/2}"/>
          <geometry>
-            <mesh filename="file://$(find arns_description)/meshes/imu.stl" scale="0.001 0.001 0.001"/>
+            <mesh filename="file:///home/ervinpicardal/robot_ws/src/arns_description/meshes/imu.stl" scale="0.001 0.001 0.001"/>
          </geometry>
       </visual>

File: arns_description/urdf/lidar.xacro (robot description, xacro)
@@ -11,5 +11,5 @@
          <origin xyz="0 0 -${lidar_height/2}"/>
          <geometry>
-            <mesh filename="file://$(find arns_description)/meshes/lidar.stl" scale="0.001 0.001 0.001"/>
+            <mesh filename="file:///home/ervinpicardal/robot_ws/src/arns_description/meshes/lidar.stl" scale="0.001 0.001 0.001"/>
          </geometry>
          <material name="black"/>

File: arns_description/urdf/robot_core.urdf.xacro (robot description, xacro)
@@ -20,5 +20,5 @@
       <visual>
          <geometry>
-            <mesh filename="file://$(find arns_description)/meshes/chassis.stl" scale="0.001 0.001 0.001"/>
+            <mesh filename="file:///home/ervinpicardal/robot_ws/src/arns_description/meshes/chassis.stl" scale="0.001 0.001 0.001"/>
          </geometry>
          <material name="white"/>
@@ -36,5 +36,5 @@
          <origin xyz="${0.350634} 0 ${0.295}" rpy="0 0 ${pi/2}"/>
          <geometry>
-            <mesh filename="file://$(find arns_description)/meshes/head.stl" scale="0.001 0.001 0.001"/>
+            <mesh filename="file:///home/ervinpicardal/robot_ws/src/arns_description/meshes/head.stl" scale="0.001 0.001 0.001"/>
          </geometry>
          <material name="lightblue"/>
@@ -50,5 +50,5 @@
          <origin xyz="${0.197125+(0.150/2)} 0 ${0.290}" rpy="0 0 0"/>
          <geometry>
-            <mesh filename="file://$(find arns_description)/meshes/head_floor.stl" scale="0.001 0.001 0.001"/>
+            <mesh filename="file:///home/ervinpicardal/robot_ws/src/arns_description/meshes/head_floor.stl" scale="0.001 0.001 0.001"/>
          </geometry>
       </visual>
@@ -63,5 +63,5 @@
       <visual>
          <geometry>
-            <mesh filename="file://$(find arns_description)/meshes/screen_case.stl" scale="0.001 0.001 0.001"/>
+            <mesh filename="file:///home/ervinpicardal/robot_ws/src/arns_description/meshes/screen_case.stl" scale="0.001 0.001 0.001"/>
          </geometry>
          <material name="lightblue"/>
@@ -86,5 +86,5 @@
       <visual>
          <geometry>
-            <mesh filename="file://$(find arns_description)/meshes/screen.stl" scale="0.001 0.001 0.001"/>
+            <mesh filename="file:///home/ervinpicardal/robot_ws/src/arns_description/meshes/screen.stl" scale="0.001 0.001 0.001"/>
          </geometry>
          <material name="black"/>
@@ -103,5 +103,5 @@
       <visual>
          <geometry>
-            <mesh filename="file://$(find arns_description)/meshes/lidar_case.stl" scale="0.001 0.001 0.001"/>
+            <mesh filename="file:///home/ervinpicardal/robot_ws/src/arns_description/meshes/lidar_case.stl" scale="0.001 0.001 0.001"/>
          </geometry>
          <material name="lightblue"/>
@@ -128,5 +128,5 @@
       <visual>
          <geometry>
-            <mesh filename="file://$(find arns_description)/meshes/left_wheel.stl" scale="0.001 0.001 0.001"/>
+            <mesh filename="file:///home/ervinpicardal/robot_ws/src/arns_description/meshes/left_wheel.stl" scale="0.001 0.001 0.001"/>
          </geometry>
          <material name="black"/>
@@ -154,5 +154,5 @@
       <visual>
          <geometry>
-            <mesh filename="file://$(find arns_description)/meshes/right_wheel.stl" scale="0.001 0.001 0.001"/>
+            <mesh filename="file:///home/ervinpicardal/robot_ws/src/arns_description/meshes/right_wheel.stl" scale="0.001 0.001 0.001"/>
          </geometry>
          <material name="black"/>

Commit message: updated rviz mesh

File: arns_description/urdf/camera.xacro (robot description, xacro)
@@ -9,5 +9,5 @@
       <visual>
          <geometry>
-            <mesh filename="file:///home/ervinpicardal/robot_ws/src/arns_description/meshes/camera.stl" scale="0.001 0.001 0.001"/>
+            <mesh filename="file:///home/display/robot_ws/src/arns/arns_description/meshes/camera.stl" scale="0.001 0.001 0.001"/>
          </geometry>
          <material name="black"/>

File: arns_description/urdf/imu.xacro (robot description, xacro)
@@ -10,5 +10,5 @@
         <origin xyz="0 0 0" rpy="0 0 ${pi/2}"/>
          <geometry>
-            <mesh filename="file:///home/ervinpicardal/robot_ws/src/arns_description/meshes/imu.stl" scale="0.001 0.001 0.001"/>
+            <mesh filename="file:///home/display/robot_ws/src/arns/arns_description/meshes/imu.stl" scale="0.001 0.001 0.001"/>
          </geometry>
       </visual>

File: arns_description/urdf/lidar.xacro (robot description, xacro)
@@ -11,5 +11,5 @@
          <origin xyz="0 0 -${lidar_height/2}"/>
          <geometry>
-            <mesh filename="file:///home/ervinpicardal/robot_ws/src/arns_description/meshes/lidar.stl" scale="0.001 0.001 0.001"/>
+            <mesh filename="file:///home/display/robot_ws/src/arns/arns_description/meshes/lidar.stl" scale="0.001 0.001 0.001"/>
          </geometry>
          <material name="black"/>

File: arns_description/urdf/robot_core.urdf.xacro (robot description, xacro)
@@ -20,5 +20,5 @@
       <visual>
          <geometry>
-            <mesh filename="file:///home/ervinpicardal/robot_ws/src/arns_description/meshes/chassis.stl" scale="0.001 0.001 0.001"/>
+            <mesh filename="file:///home/display/robot_ws/src/arns/arns_description/meshes/chassis.stl" scale="0.001 0.001 0.001"/>
          </geometry>
          <material name="white"/>
@@ -36,5 +36,5 @@
          <origin xyz="${0.350634} 0 ${0.295}" rpy="0 0 ${pi/2}"/>
          <geometry>
-            <mesh filename="file:///home/ervinpicardal/robot_ws/src/arns_description/meshes/head.stl" scale="0.001 0.001 0.001"/>
+            <mesh filename="file:///home/display/robot_ws/src/arns/arns_description/meshes/head.stl" scale="0.001 0.001 0.001"/>
          </geometry>
          <material name="lightblue"/>
@@ -50,5 +50,5 @@
          <origin xyz="${0.197125+(0.150/2)} 0 ${0.290}" rpy="0 0 0"/>
          <geometry>
-            <mesh filename="file:///home/ervinpicardal/robot_ws/src/arns_description/meshes/head_floor.stl" scale="0.001 0.001 0.001"/>
+            <mesh filename="file:///home/display/robot_ws/src/arns/arns_description/meshes/head_floor.stl" scale="0.001 0.001 0.001"/>
          </geometry>
       </visual>
@@ -63,5 +63,5 @@
       <visual>
          <geometry>
-            <mesh filename="file:///home/ervinpicardal/robot_ws/src/arns_description/meshes/screen_case.stl" scale="0.001 0.001 0.001"/>
+            <mesh filename="file:///home/display/robot_ws/src/arns/arns_description/meshes/screen_case.stl" scale="0.001 0.001 0.001"/>
          </geometry>
          <material name="lightblue"/>
@@ -86,5 +86,5 @@
       <visual>
          <geometry>
-            <mesh filename="file:///home/ervinpicardal/robot_ws/src/arns_description/meshes/screen.stl" scale="0.001 0.001 0.001"/>
+            <mesh filename="file:///home/display/robot_ws/src/arns/arns_description/meshes/screen.stl" scale="0.001 0.001 0.001"/>
          </geometry>
          <material name="black"/>
@@ -103,5 +103,5 @@
       <visual>
          <geometry>
-            <mesh filename="file:///home/ervinpicardal/robot_ws/src/arns_description/meshes/lidar_case.stl" scale="0.001 0.001 0.001"/>
+            <mesh filename="file:///home/display/robot_ws/src/arns/arns_description/meshes/lidar_case.stl" scale="0.001 0.001 0.001"/>
          </geometry>
          <material name="lightblue"/>
@@ -128,5 +128,5 @@
       <visual>
          <geometry>
-            <mesh filename="file:///home/ervinpicardal/robot_ws/src/arns_description/meshes/left_wheel.stl" scale="0.001 0.001 0.001"/>
+            <mesh filename="file:///home/display/robot_ws/src/arns/arns_description/meshes/left_wheel.stl" scale="0.001 0.001 0.001"/>
          </geometry>
          <material name="black"/>
@@ -154,5 +154,5 @@
       <visual>
          <geometry>
-            <mesh filename="file:///home/ervinpicardal/robot_ws/src/arns_description/meshes/right_wheel.stl" scale="0.001 0.001 0.001"/>
+            <mesh filename="file:///home/display/robot_ws/src/arns/arns_description/meshes/right_wheel.stl" scale="0.001 0.001 0.001"/>
          </geometry>
          <material name="black"/>

Commit message: switch models for development

File: arns_description/urdf/camera.xacro (robot description, xacro)
@@ -10,4 +10,5 @@
          <geometry>
             <mesh filename="file:///home/display/robot_ws/src/arns/arns_description/meshes/camera.stl" scale="0.001 0.001 0.001"/>
+            <mesh filename="file:///home/ervinpicardal/robot_ws/src/arns_description/meshes/camera.stl" scale="0.001 0.001 0.001"/>
          </geometry>
          <material name="black"/>

File: arns_description/urdf/imu.xacro (robot description, xacro)
@@ -10,5 +10,5 @@
         <origin xyz="0 0 0" rpy="0 0 ${pi/2}"/>
          <geometry>
-            <mesh filename="file:///home/display/robot_ws/src/arns/arns_description/meshes/imu.stl" scale="0.001 0.001 0.001"/>
+            <mesh filename="file:///home/ervinpicardal/robot_ws/src/arns_description/meshes/imu.stl" scale="0.001 0.001 0.001"/>
          </geometry>
       </visual>

File: arns_description/urdf/lidar.xacro (robot description, xacro)
@@ -12,4 +12,5 @@
          <geometry>
             <mesh filename="file:///home/display/robot_ws/src/arns/arns_description/meshes/lidar.stl" scale="0.001 0.001 0.001"/>
+            <mesh filename="file:///home/ervinpicardal/robot_ws/src/arns_description/meshes/lidar.stl" scale="0.001 0.001 0.001"/>
          </geometry>
          <material name="black"/>

File: arns_description/urdf/robot_core.urdf.xacro (robot description, xacro)
@@ -20,5 +20,6 @@
       <visual>
          <geometry>
-            <mesh filename="file:///home/display/robot_ws/src/arns/arns_description/meshes/chassis.stl" scale="0.001 0.001 0.001"/>
+            <!-- <mesh filename="file:///home/display/robot_ws/src/arns/arns_description/meshes/chassis.stl" scale="0.001 0.001 0.001"/> -->
+            <mesh filename="file:///home/ervinpicardal/robot_ws/src/arns_description/meshes/chassis.stl" scale="0.001 0.001 0.001"/>
          </geometry>
          <material name="white"/>
@@ -36,5 +37,6 @@
          <origin xyz="${0.350634} 0 ${0.295}" rpy="0 0 ${pi/2}"/>
          <geometry>
-            <mesh filename="file:///home/display/robot_ws/src/arns/arns_description/meshes/head.stl" scale="0.001 0.001 0.001"/>
+            <!-- <mesh filename="file:///home/display/robot_ws/src/arns/arns_description/meshes/head.stl" scale="0.001 0.001 0.001"/> -->
+            <mesh filename="file:///home/ervinpicardal/robot_ws/src/arns_description/meshes/head.stl" scale="0.001 0.001 0.001"/>
          </geometry>
          <material name="lightblue"/>
@@ -50,5 +52,6 @@
          <origin xyz="${0.197125+(0.150/2)} 0 ${0.290}" rpy="0 0 0"/>
          <geometry>
-            <mesh filename="file:///home/display/robot_ws/src/arns/arns_description/meshes/head_floor.stl" scale="0.001 0.001 0.001"/>
+            <!-- <mesh filename="file:///home/display/robot_ws/src/arns/arns_description/meshes/head_floor.stl" scale="0.001 0.001 0.001"/> -->
+            <mesh filename="file:///home/ervinpicardal/robot_ws/src/arns_description/meshes/head_floor.stl" scale="0.001 0.001 0.001"/>
          </geometry>
       </visual>
@@ -63,5 +66,6 @@
       <visual>
          <geometry>
-            <mesh filename="file:///home/display/robot_ws/src/arns/arns_description/meshes/screen_case.stl" scale="0.001 0.001 0.001"/>
+            <!-- <mesh filename="file:///home/display/robot_ws/src/arns/arns_description/meshes/screen_case.stl" scale="0.001 0.001 0.001"/> -->
+            <mesh filename="file:///home/ervinpicardal/robot_ws/src/arns_description/meshes/screen_case.stl" scale="0.001 0.001 0.001"/>
          </geometry>
          <material name="lightblue"/>
@@ -87,4 +91,5 @@
          <geometry>
             <mesh filename="file:///home/display/robot_ws/src/arns/arns_description/meshes/screen.stl" scale="0.001 0.001 0.001"/>
+            <mesh filename="file:///home/ervinpicardal/robot_ws/src/arns_description/meshes/screen.stl" scale="0.001 0.001 0.001"/>
          </geometry>
          <material name="black"/>
@@ -104,4 +109,5 @@
          <geometry>
             <mesh filename="file:///home/display/robot_ws/src/arns/arns_description/meshes/lidar_case.stl" scale="0.001 0.001 0.001"/>
+            <mesh filename="file:///home/ervinpicardal/robot_ws/src/arns_description/meshes/lidar_case.stl" scale="0.001 0.001 0.001"/>
          </geometry>
          <material name="lightblue"/>
@@ -129,4 +135,5 @@
          <geometry>
             <mesh filename="file:///home/display/robot_ws/src/arns/arns_description/meshes/left_wheel.stl" scale="0.001 0.001 0.001"/>
+            <mesh filename="file:///home/ervinpicardal/robot_ws/src/arns_description/meshes/left_wheel.stl" scale="0.001 0.001 0.001"/>
          </geometry>
          <material name="black"/>
@@ -155,4 +162,5 @@
          <geometry>
             <mesh filename="file:///home/display/robot_ws/src/arns/arns_description/meshes/right_wheel.stl" scale="0.001 0.001 0.001"/>
+            <mesh filename="file:///home/ervinpicardal/robot_ws/src/arns_description/meshes/right_wheel.stl" scale="0.001 0.001 0.001"/>
          </geometry>
          <material name="black"/>

Commit message: switch models for development

File: arns_description/urdf/camera.xacro (robot description, xacro)
@@ -9,5 +9,5 @@
       <visual>
          <geometry>
-            <mesh filename="file:///home/display/robot_ws/src/arns/arns_description/meshes/camera.stl" scale="0.001 0.001 0.001"/>
+            <!-- <mesh filename="file:///home/display/robot_ws/src/arns/arns_description/meshes/camera.stl" scale="0.001 0.001 0.001"/> -->
             <mesh filename="file:///home/ervinpicardal/robot_ws/src/arns_description/meshes/camera.stl" scale="0.001 0.001 0.001"/>
          </geometry>

File: arns_description/urdf/imu.xacro (robot description, xacro)
@@ -10,4 +10,5 @@
         <origin xyz="0 0 0" rpy="0 0 ${pi/2}"/>
          <geometry>
+            <!-- <mesh filename="file:///home/display/robot_ws/src/arns/arns_description/meshes/imu.stl" scale="0.001 0.001 0.001"/> -->
             <mesh filename="file:///home/ervinpicardal/robot_ws/src/arns_description/meshes/imu.stl" scale="0.001 0.001 0.001"/>
          </geometry>

File: arns_description/urdf/lidar.xacro (robot description, xacro)
@@ -11,5 +11,5 @@
          <origin xyz="0 0 -${lidar_height/2}"/>
          <geometry>
-            <mesh filename="file:///home/display/robot_ws/src/arns/arns_description/meshes/lidar.stl" scale="0.001 0.001 0.001"/>
+            <!-- <mesh filename="file:///home/display/robot_ws/src/arns/arns_description/meshes/lidar.stl" scale="0.001 0.001 0.001"/> -->
             <mesh filename="file:///home/ervinpicardal/robot_ws/src/arns_description/meshes/lidar.stl" scale="0.001 0.001 0.001"/>
          </geometry>

File: arns_description/urdf/robot_core.urdf.xacro (robot description, xacro)
@@ -90,5 +90,5 @@
       <visual>
          <geometry>
-            <mesh filename="file:///home/display/robot_ws/src/arns/arns_description/meshes/screen.stl" scale="0.001 0.001 0.001"/>
+            <!-- <mesh filename="file:///home/display/robot_ws/src/arns/arns_description/meshes/screen.stl" scale="0.001 0.001 0.001"/> -->
             <mesh filename="file:///home/ervinpicardal/robot_ws/src/arns_description/meshes/screen.stl" scale="0.001 0.001 0.001"/>
          </geometry>
@@ -108,5 +108,5 @@
       <visual>
          <geometry>
-            <mesh filename="file:///home/display/robot_ws/src/arns/arns_description/meshes/lidar_case.stl" scale="0.001 0.001 0.001"/>
+            <!-- <mesh filename="file:///home/display/robot_ws/src/arns/arns_description/meshes/lidar_case.stl" scale="0.001 0.001 0.001"/> -->
             <mesh filename="file:///home/ervinpicardal/robot_ws/src/arns_description/meshes/lidar_case.stl" scale="0.001 0.001 0.001"/>
          </geometry>
@@ -134,5 +134,5 @@
       <visual>
          <geometry>
-            <mesh filename="file:///home/display/robot_ws/src/arns/arns_description/meshes/left_wheel.stl" scale="0.001 0.001 0.001"/>
+            <!-- <mesh filename="file:///home/display/robot_ws/src/arns/arns_description/meshes/left_wheel.stl" scale="0.001 0.001 0.001"/> -->
             <mesh filename="file:///home/ervinpicardal/robot_ws/src/arns_description/meshes/left_wheel.stl" scale="0.001 0.001 0.001"/>
          </geometry>
@@ -161,5 +161,5 @@
       <visual>
          <geometry>
-            <mesh filename="file:///home/display/robot_ws/src/arns/arns_description/meshes/right_wheel.stl" scale="0.001 0.001 0.001"/>
+            <!-- <mesh filename="file:///home/display/robot_ws/src/arns/arns_description/meshes/right_wheel.stl" scale="0.001 0.001 0.001"/> -->
             <mesh filename="file:///home/ervinpicardal/robot_ws/src/arns_description/meshes/right_wheel.stl" scale="0.001 0.001 0.001"/>
          </geometry>

Commit message: added camera launch file

File: arns_description/urdf/camera.xacro (robot description, xacro)
@@ -2,5 +2,5 @@
 <robot xmlns:xacro="http://www.ros.org/wiki/xacro">
    <joint name="camera_joint" type="fixed">
-      <origin xyz="0.0 0.0 0.0" rpy="0.0 0.0 0.0"/>
+      <origin xyz="${-0.121 + 0.180 + 0.345 - 0.02} 0.0 ${chassis_height + head_height - 0.048}" rpy="0.0 0.0 0.0"/>
       <parent link="base_link"/>
       <child link="camera_link"/>
@@ -12,4 +12,41 @@
          </geometry>
       </visual>
+      <collision>
+         <origin xyz="-0.02 0.0 0.0" rpy="0.0 0.0 0.0"/>
+         <geometry>
+            <box size="0.04 0.120 0.04"/>
+         </geometry>
+      </collision>
+      <xacro:inertial_box mass="0.01" x="0.04" y="0.120" z="0.04">
+         <origin xyz="-0.02 0.0 0.0" rpy="0.0 0.0 0.0"/>
+      </xacro:inertial_box>
    </link>
+   <joint name="camera_joint_optical" type="fixed">
+      <origin xyz="0.0 0.0 0.0" rpy="-${pi/2} 0.0 -${pi/2}"/>
+      <parent link="camera_link"/>
+      <child link="camera_link_optical"/>
+   </joint>
+   <link name="camera_link_optical"></link>
+   <gazebo reference="camera_link">
+      <material>Gazebo/Red</material>
+      <sensor name="camera" type="camera">
+         <visualize>true</visualize>
+         <update_rate>30.0</update_rate>
+         <camera>
+            <horizontal_fov>1.5708</horizontal_fov>
+            <image>
+               <format>R8G8B8</format>
+               <width>640</width>
+               <height>480</height>
+            </image>
+            <clip>
+               <near>0.05</near>
+               <far>8.0</far>
+            </clip>
+         </camera>
+         <plugin name="camera_controller" filename="libgazebo_ros_camera.so">
+            <frame_name>camera_link_optical</frame_name>
+         </plugin>
+      </sensor>
+   </gazebo>
 </robot>
