Commit message: change

File: arns_description/urdf/robot.urdf.xacro (robot description, xacro)
@@ -2,5 +2,5 @@
 <robot xmlns:xacro="http://www.ros.org/wiki/xacro" name="robot_name">
    <xacro:arg name="use_ros2_control" default="true"/>
-   <xacro:arg name="sim_mode" default="false"/>
+   <!-- <xacro:arg name="sim_mode" default="false"/> -->
    <!-- Robot Physical Properties -->
    <xacro:include filename="$(find arns_description)/urdf/properties.xacro"/>

File: arns_description/urdf/ros2_control.xacro (robot description, xacro)
@@ -1,61 +1,56 @@
 <?xml version="1.0" encoding="UTF-8"?>
 <robot xmlns:xacro="http://www.ros.org/wiki/xacro">
-   <xacro:unless value="$(arg sim_mode)">
-      <ros2_control name="RealRobot" type="system">
-         <hardware>
-            <plugin>diffdrive_arduino/DiffDriveArduino</plugin>
-            <param name="left_wheel_name">left_wheel_joint</param>
-            <param name="right_wheel_name">right_wheel_joint</param>
-            <param name="loop_rate">30</param>
-            <param name="device">/dev/ttyACM0</param>
-            <param name="baud_rate">57600</param>
-            <param name="timeout">1000</param>
-            <param name="enc_counts_per_rev">2800</param>
-         </hardware>
-         <joint name="left_wheel_joint">
-            <command_interface name="velocity">
-               <param name="min">-10</param>
-               <param name="max">10</param>
-            </command_interface>
-            <state_interface name="velocity"/>
-            <state_interface name="position"/>
-         </joint>
-         <joint name="right_wheel_joint">
-            <command_interface name="velocity">
-               <param name="min">-10</param>
-               <param name="max">10</param>
-            </command_interface>
-            <state_interface name="velocity"/>
-            <state_interface name="position"/>
-         </joint>
-      </ros2_control>
-   </xacro:unless>
-   <xacro:if value="$(arg sim_mode)">
-      <ros2_control name="GazeboSystem" type="system">
-         <hardware>
-            <plugin>gazebo_ros2_control/GazeboSystem</plugin>
-         </hardware>
-         <joint name="left_wheel_joint">
-            <command_interface name="velocity">
-               <param name="min">-10</param>
-               <param name="max">10</param>
-            </command_interface>
-            <state_interface name="velocity"/>
-            <state_interface name="position"/>
-         </joint>
-         <joint name="right_wheel_joint">
-            <command_interface name="velocity">
-               <param name="min">-10</param>
-               <param name="max">10</param>
-            </command_interface>
-            <state_interface name="velocity"/>
-            <state_interface name="position"/>
-         </joint>
-      </ros2_control>
-   </xacro:if>
+   <ros2_control name="RealRobot" type="system">
+      <hardware>
+         <plugin>diffdrive_arduino/DiffDriveArduino</plugin>
+         <param name="left_wheel_name">left_wheel_joint</param>
+         <param name="right_wheel_name">right_wheel_joint</param>
+         <param name="loop_rate">30</param>
+         <param name="device">/dev/ttyACM0</param>
+         <param name="baud_rate">57600</param>
+         <param name="timeout">1000</param>
+         <param name="enc_counts_per_rev">2800</param>
+      </hardware>
+      <joint name="left_wheel_joint">
+         <command_interface name="velocity">
+            <param name="min">-10</param>
+            <param name="max">10</param>
+         </command_interface>
+         <state_interface name="velocity"/>
+         <state_interface name="position"/>
+      </joint>
+      <joint name="right_wheel_joint">
+         <command_interface name="velocity">
+            <param name="min">-10</param>
+            <param name="max">10</param>
+         </command_interface>
+         <state_interface name="velocity"/>
+         <state_interface name="position"/>
+      </joint>
+   </ros2_control>
+   <!-- <ros2_control name="GazeboSystem" type="system">
+      <hardware>
+         <plugin>gazebo_ros2_control/GazeboSystem</plugin>
+      </hardware>
+      <joint name="left_wheel_joint">
+         <command_interface name="velocity">
+            <param name="min">-10</param>
+            <param name="max">10</param>
+         </command_interface>
+         <state_interface name="velocity"/>
+         <state_interface name="position"/>
+      </joint>
+      <joint name="right_wheel_joint">
+         <command_interface name="velocity">
+            <param name="min">-10</param>
+            <param name="max">10</param>
+         </command_interface>
+         <state_interface name="velocity"/>
+         <state_interface name="position"/>
+      </joint>
+   </ros2_control>   -->
    <gazebo>
       <plugin name="gazebo_ros2_control" filename="libgazebo_ros2_control.so">
          <parameters>$(find arns_bringup)/config/controllers.yaml</parameters>
-         <parameters>$(find arns_bringup)/config/gazebo_ros2_ctl_use_sim.yaml</parameters>
       </plugin>
    </gazebo>

Commit message: added slam_toolbox

File: arns_description/urdf/robot.urdf.xacro (robot description, xacro)
@@ -2,5 +2,5 @@
 <robot xmlns:xacro="http://www.ros.org/wiki/xacro" name="robot_name">
    <xacro:arg name="use_ros2_control" default="true"/>
-   <!-- <xacro:arg name="sim_mode" default="false"/> -->
+   <xacro:arg name="sim_mode" default="false"/>
    <!-- Robot Physical Properties -->
    <xacro:include filename="$(find arns_description)/urdf/properties.xacro"/>
@@ -9,5 +9,4 @@
    <!-- ROBOT URDF -->
    <xacro:include filename="$(find arns_description)/urdf/robot_core.urdf.xacro"/>
-   <!-- initialize ros2_control -->
    <xacro:if value="$(arg use_ros2_control)">
       <!-- GAZEBO ROS2 CONTROL -->

File: arns_description/urdf/robot_core.urdf.xacro (robot description, xacro)
@@ -2,4 +2,13 @@
 <robot xmlns:xacro="http://www.ros.org/wiki/xacro">
    <link name="base_link"/>
+   <!-- BASE FOOTPRINT -->
+   <joint name="base_footprint_joint" type="fixed">
+      <parent link="base_link"/>
+      <child link="base_footprint"/>
+      <origin xyz="0 0 0" rpy="0 0 0"/>
+   </joint>
+   <link name="base_footprint">
+   </link>
+   <!-- CHASSIS -->
    <joint name="chassis_joint" type="fixed">
       <parent link="base_link"/>

File: arns_description/urdf/ros2_control.xacro (robot description, xacro)
@@ -1,5 +1,6 @@
 <?xml version="1.0" encoding="UTF-8"?>
 <robot xmlns:xacro="http://www.ros.org/wiki/xacro">
-   <ros2_control name="RealRobot" type="system">
+   <xacro:unless value="$(arg sim_mode)">
+      <ros2_control name="RealRobot" type="system">
          <hardware>
             <plugin>diffdrive_arduino/DiffDriveArduino</plugin>
@@ -29,5 +30,7 @@
          </joint>
       </ros2_control>
-   <!-- <ros2_control name="GazeboSystem" type="system">
+   </xacro:unless>
+   <xacro:if value="$(arg sim_mode)">
+   <ros2_control name="GazeboSystem" type="system">
       <hardware>
          <plugin>gazebo_ros2_control/GazeboSystem</plugin>
@@ -49,8 +52,10 @@
          <state_interface name="position"/>
       </joint>
-   </ros2_control>   -->
+   </ros2_control>
+   </xacro:if>
    <gazebo>
       <plugin name="gazebo_ros2_control" filename="libgazebo_ros2_control.so">
          <parameters>$(find arns_bringup)/config/controllers.yaml</parameters>
+         <parameters>$(find arns_bringup)/config/ros2_cnotrol_use_sim.yaml</parameters>
       </plugin>
    </gazebo>

Commit message: added ros2_control

File: arns_description/urdf/robot.urdf.xacro (robot description, xacro)
@@ -2,4 +2,5 @@
 <robot xmlns:xacro="http://www.ros.org/wiki/xacro" name="alexbot">
    <xacro:arg name="use_ros2_control" default="true"/>
+   <xacro:arg name="sim_mode" default="false"/>
    <xacro:include filename="properties.xacro"/>
    <xacro:include filename="inertial_macro.xacro"/>

File: arns_description/urdf/ros2_control.xacro (robot description, xacro)
@@ -1,28 +1,61 @@
 <?xml version="1.0" encoding="UTF-8"?>
 <robot xmlns:xacro="http://www.ros.org/wiki/xacro">
-   <ros2_control name="GazeboSystem" type="system">
-      <hardware>
-         <plugin>gazebo_ros2_control/GazeboSystem</plugin>
-      </hardware>
-      <joint name="left_wheel_joint">
-         <command_interface name="velocity">
-            <param name="min">-10</param>
-            <param name="max">10</param>
-         </command_interface>
-         <state_interface name="velocity"/>
-         <state_interface name="position"/>
-      </joint>
-      <joint name="right_wheel_joint">
-         <command_interface name="velocity">
-            <param name="min">-10</param>
-            <param name="max">10</param>
-         </command_interface>
-         <state_interface name="velocity"/>
-         <state_interface name="position"/>
-      </joint>
-   </ros2_control>
+   <xacro:unless value="$(arg sim_mode)">
+      <ros2_control name="DiffDriveSystem" type="system">
+         <hardware>
+            <plugin>diffdrive_arduino/DiffDriveArduino</plugin>
+            <param name="left_wheel_name">left_wheel_joint</param>
+            <param name="right_wheel_name">right_wheel_joint</param>
+            <param name="loop_rate">30</param>
+            <param name="device">/dev/ttyACM0</param>
+            <param name="baud_rate">57600</param>
+            <param name="timeout">1000</param>
+            <param name="enc_counts_per_rev">2800</param>
+         </hardware>
+         <joint name="left_wheel_joint">
+            <command_interface name="velocity">
+               <param name="min">-10</param>
+               <param name="max">10</param>
+            </command_interface>
+            <state_interface name="velocity"/>
+            <state_interface name="position"/>
+         </joint>
+         <joint name="right_wheel_joint">
+            <command_interface name="velocity">
+               <param name="min">-10</param>
+               <param name="max">10</param>
+            </command_interface>
+            <state_interface name="velocity"/>
+            <state_interface name="position"/>
+         </joint>
+      </ros2_control>
+   </xacro:unless>
+   <xacro:if value="$(arg sim_mode)">
+      <ros2_control name="GazeboSystem" type="system">
+         <hardware>
+            <plugin>gazebo_ros2_control/GazeboSystem</plugin>
+         </hardware>
+         <joint name="left_wheel_joint">
+            <command_interface name="velocity">
+               <param name="min">-10</param>
+               <param name="max">10</param>
+            </command_interface>
+            <state_interface name="velocity"/>
+            <state_interface name="position"/>
+         </joint>
+         <joint name="right_wheel_joint">
+            <command_interface name="velocity">
+               <param name="min">-10</param>
+               <param name="max">10</param>
+            </command_interface>
+            <state_interface name="velocity"/>
+            <state_interface name="position"/>
+         </joint>
+      </ros2_control>
+   </xacro:if>
    <gazebo>
       <plugin name="gazebo_ros2_control" filename="libgazebo_ros2_control.so">
          <parameters>$(find arns_bringup)/config/controllers.yaml</parameters>
+         <parameters>$(find arns_bringup)/config/ctl_manager_use_sim_time.yaml</parameters>
       </plugin>
    </gazebo>
