Commit message: added bringup package and lidar launch file

File: arns_description/urdf/properties.xacro (robot description, xacro)
@@ -26,4 +26,8 @@
       <xacro:property name="screen_case_width" value="0.175"/>
       <xacro:property name="screen_case_height" value="0.0298"/>
+      <!-- SCREEN -->
+      <xacro:property name="screen_length" value="0.100"/>
+      <xacro:property name="screen_width" value="0.165"/>
+      <xacro:property name="screen_height" value="0.010"/>
        <!-- LIDAR CASE -->
       <xacro:property name="lidar_case_length" value="0.110"/>
@@ -32,5 +36,5 @@
        <!-- LIDAR -->
        <xacro:property name="lidar_length" value="0.025"/>
-       <xacro:property name="lidar_radius" value="0.037"/>
+       <xacro:property name="lidar_diameter" value="0.072"/>
        <xacro:property name="lidar_mass" value="0.07"/>
       <!-- COLORS -->
@@ -48,5 +52,5 @@
      </material>
      <material name="lightblue">
-      <color rgba="${194/255} ${224/255} ${252/255} 1.0"/>
+      <color rgba="${0/255} ${141/255} ${255/255} 1.0"/>
       </material>
       <!-- MACROS -->

File: arns_description/urdf/robot.urdf.xacro (robot description, xacro)
@@ -4,4 +4,5 @@
    <xacro:include filename="$(find arns_description)/urdf/inertial_macro.xacro"/>
    <xacro:include filename="$(find arns_description)/urdf/robot_core.urdf.xacro"/>
+   <xacro:include filename="$(find arns_description)/urdf/lidar.xacro"/>
    <xacro:include filename="$(find arns_description)/urdf/gazebo_control.xacro"/>
 </robot>

File: arns_description/urdf/robot_core.urdf.xacro (robot description, xacro)
@@ -75,4 +75,73 @@
       </xacro:inertial_box>
    </link>
+   <!-- LIDAR CASE -->
+   <joint name="lidar_case_joint" type="fixed">
+      <origin xyz="-0.07 0.0 ${head_height + 0.005}" rpy="0.0 0.0 0.0"/>
+      <parent link="head_link"/>
+      <child link="lidar_case_link"/>
+   </joint>
+   <link name="lidar_case_link">
+      <visual>
+         <geometry>
+            <mesh filename="package://arns_description/meshes/lidar_case.stl" scale="0.001 0.001 0.001"/>
+         </geometry>
+         <material name="lightblue"/>
+      </visual>
+      <collision>
+         <origin xyz="-0.001 0.0 ${(lidar_case_height/2)}" rpy="0.0 0.0 0.0"/>
+         <geometry>
+            <box size="${lidar_case_length} ${lidar_case_width} ${lidar_case_height}"/>
+         </geometry>
+      </collision>
+      <xacro:inertial_box mass="0.01" x="${lidar_case_length}" y="${lidar_case_width}" z="${lidar_case_height}">
+         <origin xyz="-0.001 0.0 ${(lidar_case_height/2)}" rpy="0.0 0.0 0.0"/>
+      </xacro:inertial_box>
+   </link>
+   <!-- SCREEN CASE -->
+   <joint name="screen_case_joint" type="fixed">
+      <origin xyz="0.07 0.0 ${head_height + 0.005}" rpy="0.0 0.0 0.0"/>
+      <parent link="head_link"/>
+      <child link="screen_case_link"/>
+   </joint>
+   <link name="screen_case_link">
+      <visual>
+         <geometry>
+            <mesh filename="package://arns_description/meshes/screen_case.stl" scale="0.001 0.001 0.001"/>
+         </geometry>
+         <material name="lightblue"/>
+      </visual>
+      <collision>
+         <origin xyz="0.0 0.0 ${screen_case_height/2}" rpy="0.0 0.0 0.0"/>
+         <geometry>
+            <box size="${screen_case_length} ${screen_case_width} ${screen_case_height}"/>
+         </geometry>
+      </collision>
+      <xacro:inertial_box mass="0.01" x="${screen_case_length}" y="${screen_case_width}" z="${screen_case_height}">
+         <origin xyz="0.0 0.0 ${screen_case_height/2}" rpy="0.0 0.0 0.0"/>
+      </xacro:inertial_box>
+   </link>
+   <!-- SCREEN -->
+   <joint name="screen_joint" type="fixed">
+      <origin xyz="0.07 0.0 ${head_height + screen_case_height + 0.005}" rpy="0.0 0.0 0.0"/>
+      <parent link="head_link"/>
+      <child link="screen_link"/>
+   </joint>
+   <link name="screen_link">
+      <visual>
+         <geometry>
+            <mesh filename="package://arns_description/meshes/screen.stl" scale="0.001 0.001 0.001"/>
+         </geometry>
+         <material name="black"/>
+      </visual>
+      <collision>
+         <origin xyz="0.0 0.0 0.0" rpy="0.0 0.0 0.0"/>
+         <geometry>
+            <box size="${screen_length} ${screen_width} ${screen_height}"/>
+         </geometry>
+      </collision>
+      <xacro:inertial_box mass="0.01" x="${screen_length}" y="${screen_width}" z="${screen_height}">
+         <origin xyz="0.0 0.0 0.0" rpy="0.0 0.0 0.0"/>
+      </xacro:inertial_box>
+   </link>
    <!-- LEFT WHEEL-->
    <joint name="left_wheel_joint" type="continuous">
@@ -164,4 +233,13 @@
       <material>Gazebo/Black</material>
    </gazebo>
+   <gazebo reference="lidar_case_link">
+      <material>Gazebo/Blue</material>
+   </gazebo>
+   <gazebo reference="screen_case_link">
+      <material>Gazebo/Blue</material>
+   </gazebo>
+   <gazebo reference="screen_link">
+      <material>Gazebo/Black</material>
+   </gazebo>
    <gazebo reference="caster_wheel_link">
       <material>Gazebo/Black</material>

Commit message: fixed caster_wheel_z offset

File: arns_description/urdf/properties.xacro (robot description, xacro)
@@ -16,10 +16,10 @@
       <xacro:property name="wheel_mass" value="0.35"/>
       <xacro:property name="wheel_y_offset" value="0.120684"/>
-      <xacro:property name="wheel_z_offset" value="0.02"/>
+      <xacro:property name="wheel_z_offset" value="0.017"/>
       <!-- CASTER WHEELS -->
-      <xacro:property name="caster_wheel_radius" value="0.03"/>
+      <xacro:property name="caster_wheel_radius" value="0.033"/>
       <xacro:property name="caster_wheel_mass" value="0.4"/>
       <xacro:property name="caster_wheel_offset_x" value="0.420"/>
-      <xacro:property name="caster_wheel_offset_z" value="0.059"/>
+      <xacro:property name="caster_wheel_offset_z" value="${wheel_z_offset + (wheel_radius - caster_wheel_radius)}"/>
       <!-- SCREEN CASE -->
       <xacro:property name="screen_case_length" value="0.133"/>

File: arns_description/urdf/robot_core.urdf.xacro (robot description, xacro)
@@ -182,5 +182,4 @@
          <origin xyz="0.0 0.0 0.0" rpy="${pi/2} 0.0 0.0"/>
          <geometry>
-            <!-- <cylinder radius="${wheel_radius}" length="${wheel_length}"/> -->
             <mesh filename="package://arns_description/meshes/right_wheel.stl" scale="0.001 0.001 0.001"/>
          </geometry>
@@ -199,7 +198,7 @@
    <!-- CASTER WHEEL -->
    <joint name="caster_wheel_joint" type="fixed">
+      <origin xyz="${caster_wheel_offset_x - 0.121046} 0 -${caster_wheel_offset_z}"/>
       <parent link="base_link"/>
       <child link="caster_wheel_link"/>
-      <origin xyz="${caster_wheel_offset_x - 0.121046} 0 -0.026"/>
    </joint>
    <link name="caster_wheel_link">

Commit message: fixed wheel_seperation accuracy

File: arns_description/urdf/properties.xacro (robot description, xacro)
@@ -15,5 +15,5 @@
       <xacro:property name="wheel_length" value="0.035"/>
       <xacro:property name="wheel_mass" value="0.35"/>
-      <xacro:property name="wheel_y_offset" value="0.120684"/>
+      <xacro:property name="wheel_y_offset" value="0.1225"/>
       <xacro:property name="wheel_z_offset" value="0.017"/>
       <!-- CASTER WHEELS -->
