Commit message: added ros2_control for simulation

File: arns_description/urdf/gazebo_control.xacro (robot description, xacro)
@@ -6,6 +6,6 @@
          <left_joint>left_wheel_joint</left_joint>
          <right_joint>right_wheel_joint</right_joint>
-         <wheel_separation>0.120684</wheel_separation>
-         <wheel_diameter>0.08</wheel_diameter>
+         <wheel_separation>0.241368</wheel_separation>
+         <wheel_diameter>0.0795</wheel_diameter>
          <!-- limits -->
          <max_wheel_torque>20</max_wheel_torque>

File: arns_description/urdf/robot.urdf.xacro (robot description, xacro)
@@ -1,9 +1,15 @@
 <?xml version="1.0" encoding="UTF-8"?>
 <robot xmlns:xacro="http://www.ros.org/wiki/xacro" name="alexbot">
-   <xacro:include filename="$(find arns_description)/urdf/properties.xacro"/>
-   <xacro:include filename="$(find arns_description)/urdf/inertial_macro.xacro"/>
-   <xacro:include filename="$(find arns_description)/urdf/robot_core.urdf.xacro"/>
-   <xacro:include filename="$(find arns_description)/urdf/lidar.xacro"/>
-   <xacro:include filename="$(find arns_description)/urdf/camera.xacro"/>
-   <xacro:include filename="$(find arns_description)/urdf/gazebo_control.xacro"/>
+   <xacro:arg name="use_ros2_control" default="true"/>
+   <xacro:include filename="properties.xacro"/>
+   <xacro:include filename="inertial_macro.xacro"/>
+   <xacro:include filename="robot_core.urdf.xacro"/>
+   <xacro:if value="$(arg use_ros2_control)">
+      <xacro:include filename="ros2_control.xacro"/>
+   </xacro:if>
+   <xacro:unless value="$(arg use_ros2_control)">
+      <xacro:include filename="gazebo_control.xacro"/>
+   </xacro:unless>
+   <xacro:include filename="lidar.xacro"/>
+   <xacro:include filename="camera.xacro"/>
 </robot>

File: arns_description/urdf/robot_core.urdf.xacro (robot description, xacro)
@@ -150,5 +150,5 @@
       <child link="left_wheel_link"/>
       <axis xyz="0.0 0.0 1"/>
-      <dynamics damping="0.7" friction="0.1" />
+      <!-- <dynamics damping="0.7" friction="0.1" /> -->
    </joint>
    <link name="left_wheel_link">
@@ -156,5 +156,4 @@
          <origin xyz="0.0 0.0 0.0" rpy="-${pi/2} 0.0 0.0"/>
          <geometry>
-            <!-- <cylinder radius="${wheel_radius}" length="${wheel_length}"/> -->
             <mesh filename="package://arns_description/meshes/left_wheel.stl" scale="0.001 0.001 0.001"/>
          </geometry>
@@ -164,5 +163,5 @@
          <origin xyz="0.0 0.0 0.0" rpy="0.0 0.0 0.0"/>
          <geometry>
-            <cylinder radius="${wheel_radius + 0.002}" length="${wheel_length}"/>
+            <sphere radius="${wheel_radius}"/>
          </geometry>
       </collision>
@@ -177,5 +176,5 @@
       <child link="right_wheel_link"/>
       <axis xyz="0.0 0.0 -1"/>
-      <dynamics damping="0.7" friction="0.1" />
+      <!-- <dynamics damping="0.7" friction="0.1" /> -->
    </joint>
    <link name="right_wheel_link">
@@ -191,5 +190,5 @@
          <origin xyz="0.0 0.0 0.0" rpy="0.0 0.0 0.0"/>
          <geometry>
-            <cylinder radius="${wheel_radius + 0.002}" length="${wheel_length}"/>
+            <sphere radius="${wheel_radius}"/>
          </geometry>
       </collision>

Commit message: fixed ros2_control configs

File: arns_description/urdf/gazebo_control.xacro (robot description, xacro)
@@ -6,5 +6,5 @@
          <left_joint>left_wheel_joint</left_joint>
          <right_joint>right_wheel_joint</right_joint>
-         <wheel_separation>0.241368</wheel_separation>
+         <wheel_separation>0.232</wheel_separation>
          <wheel_diameter>0.0795</wheel_diameter>
          <!-- limits -->

File: arns_description/urdf/properties.xacro (robot description, xacro)
@@ -15,5 +15,5 @@
       <xacro:property name="wheel_length" value="0.035"/>
       <xacro:property name="wheel_mass" value="0.35"/>
-      <xacro:property name="wheel_y_offset" value="0.1225"/>
+      <xacro:property name="wheel_y_offset" value="0.11815"/>
       <xacro:property name="wheel_z_offset" value="0.017"/>
       <!-- CASTER WHEELS -->
