Commit message: IMU added

File: arns_description/urdf/imu.xacro (robot description, xacro)
@@ -21,4 +21,5 @@
    </link>
    <gazebo reference="imu_link">
+    <material>Gazebo/Red</material>
       <sensor name="bno055_imu" type="imu">
        <plugin name="imu_controller" filename="libgazebo_ros_imu_sensor.so">

File: arns_description/urdf/robot.urdf.xacro (robot description, xacro)
@@ -18,6 +18,6 @@
    </xacro:unless>
    <!-- Sensors -->
+   <xacro:include filename="$(find arns_description)/urdf/imu.xacro"/>
    <xacro:include filename="$(find arns_description)/urdf/lidar.xacro"/>
    <xacro:include filename="$(find arns_description)/urdf/camera.xacro"/>
-   <!-- <xacro:include filename="$(find arns_description)/urdf/imu.xacro"/> -->
 </robot>

Commit message: new map

File: arns_description/urdf/imu.xacro (robot description, xacro)
@@ -21,20 +21,79 @@
    </link>
    <gazebo reference="imu_link">
-    <material>Gazebo/Red</material>
-    <gravity>true</gravity>
+      <material>Gazebo/Red</material>
       <sensor name="bno055_imu" type="imu">
-       <always_on>true</always_on>
-       <update_rate>100</update_rate>
-       <visualize>true</visualize>
-       <plugin name="imu_controller" filename="libgazebo_ros_imu_sensor.so">
-          <ros>
-            <remapping>~/out:=imu_broadcaster/imu</remapping>
-          </ros>
-         <initial_orientation_as_reference>false</initial_orientation_as_reference>
-         <gaussianNoise>0.0</gaussianNoise>
-         <xyzOffset>0 0 0</xyzOffset>
-         <rpyOffset>0 0 0</rpyOffset>
-       </plugin>
+         <always_on>true</always_on>
+         <update_rate>100</update_rate>
+         <visualize>true</visualize>
+         <plugin name="imu_controller" filename="libgazebo_ros_imu_sensor.so">
+            <frame_name>imu_link</frame_name>
+            <ros>
+               <remapping>~/out:=imu_broadcaster/imu</remapping>
+            </ros>
+            <initial_orientation_as_reference>false</initial_orientation_as_reference>
+         </plugin>
+         <imu>
+            <angular_velocity>
+               <x>
+               <noise type="gaussian">
+                  <mean>0.0</mean>
+                  <stddev>2e-4</stddev>
+               </noise>
+               </x>
+               <y>
+               <noise type="gaussian">
+                  <mean>0.0</mean>
+                  <stddev>2e-4</stddev>
+               </noise>
+               </y>
+               <z>
+               <noise type="gaussian">
+                  <mean>0.0</mean>
+                  <stddev>2e-4</stddev>
+               </noise>
+               </z>
+            </angular_velocity>
+            <linear_acceleration>
+               <x>
+               <noise type="gaussian">
+                  <mean>0.0</mean>
+                  <stddev>1.7e-2</stddev>
+               </noise>
+               </x>
+               <y>
+               <noise type="gaussian">
+                  <mean>0.0</mean>
+                  <stddev>1.7e-2</stddev>
+               </noise>
+               </y>
+               <z>
+               <noise type="gaussian">
+                  <mean>0.0</mean>
+                  <stddev>1.7e-2</stddev>
+               </noise>
+               </z>
+            </linear_acceleration>
+            <orientation>
+               <x>
+               <noise type="gaussian">
+                  <mean>0.0</mean>
+                  <stddev>2e-3</stddev>
+                  </noise>
+               </x>
+               <y>
+                  <noise type="gaussian">
+                  <mean>0.0</mean>
+                  <stddev>2e-3</stddev>
+                  </noise>
+               </y>
+               <z>
+                  <noise type="gaussian">
+                  <mean>0.0</mean>
+                  <stddev>2e-3</stddev>
+                  </noise>
+               </z>
+            </orientation>
+         </imu>
       </sensor>
-    </gazebo>
+</gazebo>
 </robot>

Commit message: updated

File: arns_description/urdf/imu.xacro (robot description, xacro)
@@ -10,5 +10,4 @@
         <origin xyz="0 0 0" rpy="0 0 ${pi/2}"/>
          <geometry>
-            <!-- <mesh filename="file:///home/display/robot_ws/src/arns/arns_description/meshes/imu.stl" scale="0.001 0.001 0.001"/> -->
             <mesh filename="file:///home/ervinpicardal/robot_ws/src/arns_description/meshes/imu.stl" scale="0.001 0.001 0.001"/>
          </geometry>

File: arns_description/urdf/properties.xacro (robot description, xacro)
@@ -38,4 +38,6 @@
        <xacro:property name="lidar_diameter" value="0.072"/>
        <xacro:property name="lidar_mass" value="0.07"/>
+       <!-- center at base_link from chassis -->
+       <xacro:property name="move_to_center" value="${0.180 + 0.020}"/>
       <!-- COLORS -->
       <material name="white">

File: arns_description/urdf/robot_core.urdf.xacro (robot description, xacro)
@@ -1,7 +1,24 @@
 <?xml version="1.0" encoding="UTF-8"?>
 <robot xmlns:xacro="http://www.ros.org/wiki/xacro">
+   <!-- BASE FOOTPRINT -->
+   <link name="base_footprint">
+   </link>
+   <!-- BASE LINK -->
+   <joint name="base_joint" type="fixed">
+      <origin xyz="0 0 -${wheel_z_offset + wheel_radius}" rpy="0 0 0"/>
+      <parent link="base_link"/>
+      <child link="base_footprint"/>
+   </joint>
    <link name="base_link">
-      <visual>
-         <origin xyz="-0.121 0.0 0.0" rpy="0.0 0.0 0.0"/>
+   </link>
+   <!-- CHASSIS_LINK -->
+   <joint name="chassis_joint" type="fixed">
+      <origin xyz="-0.121 0.0 0.0" rpy="0.0 0.0 0.0"/>
+      <parent link="base_link"/>
+      <child link="chassis_link"/>
+   </joint>
+   <link name="chassis_link">
+      <visual>
+         <origin xyz="0.0 0.0 0.0" rpy="0.0 0.0 0.0"/>
         <geometry>
             <mesh filename="package://arns_description/meshes/chassis.stl" scale="0.001 0.001 0.001"/>
@@ -10,11 +27,26 @@
       </visual>
       <collision>
-         <origin xyz="${(chassis_length/2)-0.121} 0.0 ${chassis_height/2}" rpy="0.0 0.0 0.0"/>
+         <origin xyz="${chassis_length/2} 0.0 ${chassis_height/2}" rpy="0.0 0.0 0.0"/>
          <geometry>
             <box size="${chassis_length} ${chassis_width} ${chassis_height}"/>
          </geometry>
       </collision>
+      <!-- Head -->
+      <visual>
+         <origin xyz="${0.180 + (0.345/2) - 0.005} 0.0 ${chassis_height - 0.0134}" rpy="0.0 0.0 ${pi/2}"/>
+         <geometry>
+            <mesh filename="package://arns_description/meshes/head.stl" scale="0.001 0.001 0.001"/>
+         </geometry>
+         <material name="white"/>
+      </visual>
+      <collision>
+         <origin xyz="${(head_length/2) + move_to_center - 0.0025} 0 ${(head_height/2) + chassis_height}" rpy="0 0 0"/>
+         <geometry>
+            <box size="${head_length} ${head_width} ${head_height}"/>
+         </geometry>
+      </collision>
+      <!-- Head Floors -->
       <visual name="head_floor1_visual">
-         <origin xyz="0.150 0.0 ${chassis_height - 0.020}" rpy="0.0 0.0 0.0"/>
+         <origin xyz="${0.075 + move_to_center} 0.0 ${chassis_height - 0.020}" rpy="0.0 0.0 0.0"/>
          <geometry>
             <mesh filename="package://arns_description/meshes/head_floor.stl" scale="0.001 0.001 0.001"/>
@@ -22,5 +54,5 @@
       </visual>
       <collision name="head_floor1_collision">
-         <origin xyz="0.150 0.0 ${chassis_height - 0.015}" rpy="0.0 0.0 0.0"/>
+         <origin xyz="${0.075 + move_to_center} 0.0 ${chassis_height - 0.015}" rpy="0.0 0.0 0.0"/>
          <geometry>
             <box size="0.150 0.260 0.020"/>
@@ -28,5 +60,5 @@
       </collision>
       <visual name="head_floor2_visual">
-         <origin xyz="0.3 0.0 ${chassis_height - 0.020}" rpy="0.0 0.0 0.0"/>
+         <origin xyz="${0.075 + move_to_center + 0.150} 0.0 ${chassis_height - 0.020}" rpy="0.0 0.0 0.0"/>
          <geometry>
             <mesh filename="package://arns_description/meshes/head_floor.stl" scale="0.001 0.001 0.001"/>
@@ -34,112 +66,38 @@
       </visual>
       <collision name="head_floor2_collision">
-         <origin xyz="0.3 0.0 ${chassis_height - 0.015}" rpy="0.0 0.0 0.0"/>
+         <origin xyz="${0.075 + move_to_center + 0.150} 0.0 ${chassis_height - 0.015}" rpy="0.0 0.0 0.0"/>
          <geometry>
             <box size="0.150 0.260 0.020"/>
          </geometry>
       </collision>
+      <!-- Lidar Case -->
+      <visual>
+         <origin xyz="${(lidar_case_length/2) + move_to_center + 0.0228} 0.0 ${chassis_height + head_height - 0.008}" rpy="0.0 0.0 0.0"/>
+         <geometry>
+            <mesh filename="package://arns_description/meshes/lidar_case.stl" scale="0.001 0.001 0.001"/>
+         </geometry>
+         <material name="lightblue"/>
+      </visual>
+      <collision>
+         <origin xyz="${(lidar_case_length/2) + move_to_center + 0.0228} 0.0 ${chassis_height + head_height + (lidar_case_height/2) - 0.008}" rpy="0.0 0.0 0.0"/>
+         <geometry>
+            <box size="${lidar_case_length} ${lidar_case_width} ${lidar_case_height}"/>
+         </geometry>
+      </collision>
+      <!-- Screen Case -->
+      <visual>
+         <origin xyz="${(screen_case_length/2) + move_to_center - 0.0025 + 0.150 + 0.0035} 0.0 ${chassis_height + head_height - 0.008}" rpy="0.0 0.0 0.0"/>
+         <geometry>
+            <mesh filename="package://arns_description/meshes/screen_case.stl" scale="0.001 0.001 0.001"/>
+         </geometry>
+      </visual>
+      <collision>
+         <origin xyz="${(screen_case_length/2) + move_to_center - 0.0025 + 0.150 + 0.0035} 0.0 ${(screen_case_height/2) + chassis_height + head_height - 0.008}" rpy="0.0 0.0 0.0"/>
+         <geometry>
+            <box size="${screen_case_length} ${screen_case_width} ${screen_case_height}"/>
+         </geometry>
+      </collision>
       <xacro:inertial_box mass="${chassis_mass}" x="${chassis_length}" y="${chassis_width}" z="${chassis_height}">
-         <origin xyz="${(chassis_length/2)-0.121} 0.0 ${chassis_height/2}" rpy="0.0 0.0 0.0"/>
-      </xacro:inertial_box>
-   </link>
-   <link name="base_footprint">
-   </link>
-   <!-- CHASSIS -->
-   <joint name="base_joint" type="fixed">
-      <origin xyz="0 0 ${wheel_z_offset + wheel_radius}" rpy="0 0 0"/>
-      <parent link="base_footprint"/>
-      <child link="base_link"/>
-   </joint>
-   <!-- HEAD -->
-   <joint name="head_joint" type="fixed">
-      <origin xyz="${-0.121 + 0.180 + (0.345/2) - 0.005} 0.0 ${chassis_height - 0.0134}" rpy="0.0 0.0 0.0"/>
-      <parent link="base_link"/>
-      <child link="head_link"/>
-   </joint>
-   <link name="head_link">
-      <visual>
-         <origin xyz="0.0 0.0 0.0" rpy="0.0 0.0 ${pi/2}"/>
-         <geometry>
-            <mesh filename="package://arns_description/meshes/head.stl" scale="0.001 0.001 0.001"/>
-         </geometry>
-         <material name="white"/>
-      </visual>
-      <collision>
-         <origin xyz="0.005 0 ${(head_height/2) + 0.005}" rpy="0.0 0.0 0.0"/>
-         <geometry>
-            <box size="${head_length + 0.040} ${head_width} ${head_height}"/>
-         </geometry>
-      </collision>
-      <xacro:inertial_box mass="${head_mass}" x="${head_width}" y="${head_length}" z="${head_height}">
-         <origin xyz="${0.005} 0.0 ${(head_height/2) + 0.005}" rpy="0.0 0.0 ${pi/2}"/>
-      </xacro:inertial_box>
-   </link>
-   <!-- LIDAR CASE -->
-   <joint name="lidar_case_joint" type="fixed">
-      <origin xyz="-0.07 0.0 ${head_height + 0.005}" rpy="0.0 0.0 0.0"/>
-      <parent link="head_link"/>
-      <child link="lidar_case_link"/>
-   </joint>
-   <link name="lidar_case_link">
-      <visual>
-         <geometry>
-            <mesh filename="package://arns_description/meshes/lidar_case.stl" scale="0.001 0.001 0.001"/>
-         </geometry>
-         <material name="lightblue"/>
-      </visual>
-      <collision>
-         <origin xyz="-0.001 0.0 ${(lidar_case_height/2)}" rpy="0.0 0.0 0.0"/>
-         <geometry>
-            <box size="${lidar_case_length} ${lidar_case_width} ${lidar_case_height}"/>
-         </geometry>
-      </collision>
-      <xacro:inertial_box mass="0.01" x="${lidar_case_length}" y="${lidar_case_width}" z="${lidar_case_height}">
-         <origin xyz="-0.001 0.0 ${(lidar_case_height/2)}" rpy="0.0 0.0 0.0"/>
-      </xacro:inertial_box>
-   </link>
-   <!-- SCREEN CASE -->
-   <joint name="screen_case_joint" type="fixed">
-      <origin xyz="0.07 0.0 ${head_height + 0.005}" rpy="0.0 0.0 0.0"/>
-      <parent link="head_link"/>
-      <child link="screen_case_link"/>
-   </joint>
-   <link name="screen_case_link">
-      <visual>
-         <geometry>
-            <mesh filename="package://arns_description/meshes/screen_case.stl" scale="0.001 0.001 0.001"/>
-         </geometry>
-         <material name="lightblue"/>
-      </visual>
-      <collision>
-         <origin xyz="0.0 0.0 ${screen_case_height/2}" rpy="0.0 0.0 0.0"/>
-         <geometry>
-            <box size="${screen_case_length} ${screen_case_width} ${screen_case_height}"/>
-         </geometry>
-      </collision>
-      <xacro:inertial_box mass="0.01" x="${screen_case_length}" y="${screen_case_width}" z="${screen_case_height}">
-         <origin xyz="0.0 0.0 ${screen_case_height/2}" rpy="0.0 0.0 0.0"/>
-      </xacro:inertial_box>
-   </link>
-   <!-- SCREEN -->
-   <joint name="screen_joint" type="fixed">
-      <origin xyz="0.07 0.0 ${head_height + screen_case_height + 0.005}" rpy="0.0 0.0 0.0"/>
-      <parent link="head_link"/>
-      <child link="screen_link"/>
-   </joint>
-   <link name="screen_link">
-      <visual>
-         <geometry>
-            <mesh filename="package://arns_description/meshes/screen.stl" scale="0.001 0.001 0.001"/>
-         </geometry>
-         <material name="black"/>
-      </visual>
-      <collision>
-         <origin xyz="0.0 0.0 0.0" rpy="0.0 0.0 0.0"/>
-         <geometry>
-            <box size="${screen_length} ${screen_width} ${screen_height}"/>
-         </geometry>
-      </collision>
-      <xacro:inertial_box mass="0.01" x="${screen_length}" y="${screen_width}" z="${screen_height}">
-         <origin xyz="0.0 0.0 0.0" rpy="0.0 0.0 0.0"/>
+         <origin xyz="${chassis_length/2} 0.0 ${chassis_height/2}" rpy="0.0 0.0 0.0"/>
       </xacro:inertial_box>
    </link>
@@ -219,10 +177,10 @@
       </xacro:inertial_sphere>
    </link>
-   <gazebo reference="base_link">
+   <gazebo reference="chassis_link">
       <material>Gazebo/White</material>
    </gazebo>
-   <gazebo reference="head_link">
+   <!-- <gazebo reference="head_link">
       <material>Gazebo/White</material>
-   </gazebo>
+   </gazebo> -->
    <gazebo reference="left_wheel_link">
       <material>Gazebo/Black</material>
@@ -231,4 +189,5 @@
       <material>Gazebo/Black</material>
    </gazebo>
+<!--
    <gazebo reference="lidar_case_link">
       <material>Gazebo/Blue</material>
@@ -239,5 +198,5 @@
    <gazebo reference="screen_link">
       <material>Gazebo/Black</material>
-   </gazebo>
+   </gazebo> -->
    <gazebo reference="caster_wheel_link">
       <material>Gazebo/Black</material>
